File: HeadphoneAmplifier_CMoy.kicad_sch (KiCad schematic)
At the start: 0 parts

Commit message: Reference design: https://tangentsoft.com/audio/cmoy/misc/cmoy-tangent-sch.pdf
Parts:
- added BT1, BT2: 9V, symbol Device:Battery_Cell
- added C1, C2: 220uF, symbol Device:C_US
- added C3, C4: 0.1uF, symbol Device:C
- added D1: LED, symbol Device:LED
- added J1, J2: AudioJack3, symbol Connector_Audio:AudioJack3
- added R1, R10, R11, R8, R9: 10K, symbol Device:R
- added R2, R3: 4.7K, symbol Device:R
- added R4, R5: 100K, symbol Device:R
- added R6, R7: 1K, symbol Device:R
- added RV1: 10K, symbol Device:R_Potentiometer_Dual
- added SW1: SW_SPST, symbol Switch:SW_SPST
- added U1: NE5532, symbol Amplifier_Operational:NE5532
Connections:
- new net: C3.2, R4.1, U1.3 (+)
- new net: C4.2, R5.1, U1.5 (+)
- new net: R7.1, R9.1, U1.6 (-)
- new net: R11.1, U1.7
- new net: D1.2 (A), R1.2
- new net: J1.R, RV1.1
- new net: J1.T, RV1.4
- new net: BT1.2 (-), BT2.1 (+)
- new net: BT1.1 (+), SW1.1 (A)
- new net: R6.1, R8.1, U1.2 (-)
- new net: R10.1, U1.1
- new net +9V: C1.1, R1.1, R2.1, SW1.2 (B), U1.8 (V+)
- new net -9V: BT2.2 (-), C2.2, D1.1 (K), R3.2, U1.4 (V-)
- new net GND: C1.2, C2.1, J1.S, J2.S, R2.2, R3.1, R4.2, R5.2, R6.2, R7.2, RV1.3, RV1.6
- new net IN Left: C4.1, RV1.5
- new net IN Right: C3.1, RV1.2
- new net OUT Left: J2.T, R11.2, R9.2
- new net OUT Right: J2.R, R10.2, R8.2
Other:
- note added: "Power Section"
